File: wisleep_cad/wisleep/wisleep_dbg_revB.sch (EAGLE design)
At the start: 3 parts

Commit message: cad: rev B to fab
Parts:
- removed U$2: M04X2, SparkFun-Connectors:M04X2
- added JP2: FTDI_DEVICE, SparkFun-Connectors:FTDI_DEVICE
- added JP4: M05X2PTH, SparkFun-Connectors:M05X2PTH
Connections:
- new net WRX: JP2.RXI, JP4.10
- new net WTX: JP2.TXO, JP4.9
- net 3.3V: now also JP4.1; no longer U$2.1
- net DBG_IO: now also JP2.DTR, JP4.4; no longer JP1.DTR, U$2.4
- net GND: now also JP2.GND, JP4.7; no longer U$2.7
- net RST: now also JP4.2; no longer U$2.2
- net SWCLK: now also JP4.8; no longer U$2.8
- net SWDIO: now also JP4.6; no longer U$2.6
- net USART_RX: now also JP4.5; no longer U$2.5
- net USART_TX: now also JP4.3; no longer U$2.3
Changed lines of the file:
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@@
 <setting verticaltext="up"/>
 </settings>
-<grid distance="0.1" unitdist="inch" unit="inch" style="lines" multiple="1" display="no" altdistance="0.01" altunitdist="inch" altunit="inch"/>
+<grid distance="0.05" unitdist="inch" unit="inch" style="lines" multiple="1" display="no" altdistance="0.01" altunitdist="inch" altunit="inch"/>
 <layers>
 <layer number="1" name="Top" color="4" fill="1" visible="no" active="no"/>
@@
 <parts>
 <part name="JP1" library="SparkFun-Connectors" deviceset="FTDI_DEVICE" device=""/>
-<part name="U$2" library="SparkFun-Connectors" deviceset="M04X2" device=""/>
 <part name="GND5" library="SparkFun-Aesthetics" deviceset="GND" device=""/>
 <part name="SUPPLY2" library="SparkFun-Aesthetics" deviceset="3.3V" device=""/>
@@
 <part name="SUPPLY1" library="SparkFun-Aesthetics" deviceset="3.3V" device=""/>
 <part name="JP3" library="SparkFun-Connectors" deviceset="M05" device="LOCK"/>
+<part name="JP2" library="SparkFun-Connectors" deviceset="FTDI_DEVICE" device=""/>
+<part name="JP4" library="SparkFun-Connectors" deviceset="M05X2" device="PTH"/>
+<part name="GND3" library="SparkFun-Aesthetics" deviceset="GND" device=""/>
 </parts>
 <sheets>
@@
 <instances>
 <instance part="JP1" gate="G$1" x="119.38" y="43.18"/>
-<instance part="U$2" gate="G$1" x="69.85" y="40.64"/>
-<instance part="GND5" gate="1" x="57.15" y="33.02"/>
+<instance part="GND5" gate="1" x="59.69" y="27.94"/>
 <instance part="SUPPLY2" gate="G$1" x="57.15" y="48.26"/>
 <instance part="GND1" gate="1" x="25.4" y="27.94"/>
@@
 <instance part="SUPPLY1" gate="G$1" x="25.4" y="45.72"/>
 <instance part="JP3" gate="G$1" x="7.62" y="38.1"/>
+<instance part="JP2" gate="G$1" x="119.38" y="15.24"/>
+<instance part="JP4" gate="G$1" x="69.85" y="40.64"/>
+<instance part="GND3" gate="1" x="109.22" y="2.54"/>
 </instances>
 <busses>
@@
 <net name="GND" class="0">
 <segment>
-<pinref part="U$2" gate="G$1" pin="7"/>
-<wire x1="62.23" y1="38.1" x2="57.15" y2="38.1" width="0.127" layer="91"/>
-<wire x1="57.15" y1="38.1" x2="57.15" y2="35.56" width="0.127" layer="91"/>
+<wire x1="62.23" y1="38.1" x2="59.69" y2="38.1" width="0.127" layer="91"/>
+<wire x1="59.69" y1="38.1" x2="59.69" y2="30.48" width="0.127" layer="91"/>
 <pinref part="GND5" gate="1" pin="GND"/>
+<pinref part="JP4" gate="G$1" pin="7"/>
 </segment>
 <segment>
@@
 <pinref part="GND2" gate="1" pin="GND"/>
 </segment>
+<segment>
+<pinref part="JP2" gate="G$1" pin="GND"/>
+<wire x1="114.3" y1="7.62" x2="109.22" y2="7.62" width="0.127" layer="91"/>
+<wire x1="109.22" y1="7.62" x2="109.22" y2="5.08" width="0.127" layer="91"/>
+<pinref part="GND3" gate="1" pin="GND"/>
+</segment>
 </net>
 <net name="3.3V" class="0">
 <segment>
-<pinref part="U$2" gate="G$1" pin="1"/>
 <wire x1="62.23" y1="45.72" x2="57.15" y2="45.72" width="0.127" layer="91"/>
 <wire x1="57.15" y1="45.72" x2="57.15" y2="48.26" width="0.127" layer="91"/>
 <pinref part="SUPPLY2" gate="G$1" pin="3.3V"/>
+<pinref part="JP4" gate="G$1" pin="1"/>
 </segment>
 <segment>
@@
 <net name="RST" class="0">
 <segment>
-<pinref part="U$2" gate="G$1" pin="2"/>
 <wire x1="77.47" y1="45.72" x2="82.55" y2="45.72" width="0.127" layer="91"/>
 <label x="82.55" y="45.72" size="1.778" layer="95"/>
+<pinref part="JP4" gate="G$1" pin="2"/>
 </segment>
 <segment>
@@
 <net name="USART_TX" class="0">
 <segment>
-<pinref part="U$2" gate="G$1" pin="3"/>
 <wire x1="62.23" y1="43.18" x2="57.15" y2="43.18" width="0.127" layer="91"/>
 <label x="44.45" y="43.18" size="1.778" layer="95"/>
+<pinref part="JP4" gate="G$1" pin="3"/>
 </segment>
 <segment>
@@
 <net name="USART_RX" class="0">
 <segment>
-<pinref part="U$2" gate="G$1" pin="5"/>
 <wire x1="62.23" y1="40.64" x2="57.15" y2="40.64" width="0.127" layer="91"/>
 <label x="44.45" y="40.64" size="1.778" layer="95"/>
+<pinref part="JP4" gate="G$1" pin="5"/>
 </segment>
 <segment>
@@
 <net name="SWDIO" class="0">
 <segment>
-<pinref part="U$2" gate="G$1" pin="6"/>
 <wire x1="77.47" y1="40.64" x2="82.55" y2="40.64" width="0.127" layer="91"/>
 <label x="82.55" y="40.64" size="1.778" layer="95"/>
+<pinref part="JP4" gate="G$1" pin="6"/>
 </segment>
 <segment>
@@
 <net name="SWCLK" class="0">
 <segment>
-<pinref part="U$2" gate="G$1" pin="8"/>
 <wire x1="77.47" y1="38.1" x2="82.55" y2="38.1" width="0.127" layer="91"/>
 <label x="82.55" y="38.1" size="1.778" layer="95"/>
+<pinref part="JP4" gate="G$1" pin="8"/>
 </segment>
 <segment>
@@
 <net name="DBG_IO" class="0">
 <segment>
-<pinref part="U$2" gate="G$1" pin="4"/>
 <wire x1="77.47" y1="43.18" x2="82.55" y2="43.18" width="0.127" layer="91"/>
 <label x="82.55" y="43.18" size="1.778" layer="95"/>
-</segment>
-<segment>
-<pinref part="JP1" gate="G$1" pin="DTR"/>
-<wire x1="114.3" y1="48.26" x2="109.22" y2="48.26" width="0.127" layer="91"/>
-<label x="96.52" y="48.26" size="1.778" layer="95"/>
-</segment>
-</net>
+<pinref part="JP4" gate="G$1" pin="4"/>
+</segment>
+<segment>
+<pinref part="JP2" gate="G$1" pin="DTR"/>
+<wire x1="114.3" y1="20.32" x2="109.22" y2="20.32" width="0.127" layer="91"/>
+<label x="97.79" y="20.32" size="1.778" layer="95"/>
+</segment>
+</net>
+<net name="WTX" class="0">
+<segment>
+<pinref part="JP2" gate="G$1" pin="TXO"/>
+<wire x1="114.3" y1="17.78" x2="109.22" y2="17.78" width="0.127" layer="91"/>
+<label x="97.79" y="17.78" size="1.778" layer="95"/>
+</segment>
+<segment>
+<pinref part="JP4" gate="G$1" pin="9"/>
+<wire x1="62.23" y1="35.56" x2="57.15" y2="35.56" width="0.127" layer="91"/>
+<label x="44.45" y="35.56" size="1.778" layer="95"/>
+</segment>
+</net>
+<net name="WRX" class="0">
+<segment>
+<pinref part="JP2" gate="G$1" pin="RXI"/>
+<wire x1="114.3" y1="15.24" x2="109.22" y2="15.24" width="0.127" layer="91"/>
+<label x="97.79" y="15.24" size="1.778" layer="95"/>
+</segment>
+<segment>
+<pinref part="JP4" gate="G$1" pin="10"/>
+<wire x1="77.47" y1="35.56" x2="82.55" y2="35.56" width="0.127" layer="91"/>
+<label x="82.55" y="35.56" size="1.778" layer="95"/>
+</segment>
+</net>
