File: wisleep_cad/wisleep/wisleep_revB.brd (EAGLE design)
At the start: 52.1 x 54 mm, 55 parts, among them IC1 STM32F10XCXT6, X1 8MHz, X2 32kHz, X3 USB-MINIB

Commit message: cad: rev B to fab
Parts:
- removed U$1: M04X2, SparkFun-Connectors:2X4
- added C20: (no value), SparkFun-Capacitors:EIA6032
- added JP5: M05X2PTH, SparkFun-Connectors:AVR_ICSP
- moved C8 4.61 mm to (24.0, 42.8), flipped to the bottom
- moved R14 3.82 mm to (26.5, 43.0), turned to 270 degrees
- moved NTC1 2.26 mm to (29.5, 43.0), turned to 90 degrees
- moved R13 1.90 mm to (28.0, 43.0), turned to 270 degrees
Connections:
- removed net N$26: IC1.41
- new net PB3: IC1.39
- net 3.3V: now also JP5.1; no longer U$1.1
- net 5V_ENA: now also IC1.41; no longer IC1.39
- net DBG_IO: now also JP5.4; no longer U$1.4
- net GND: now also C20.P$2, JP5.7; no longer U$1.7
- net N$16: now also C3.1
- net N$3: no longer C3.1
- net POWDC: now also C20.P$1
- net RST: now also JP5.2; no longer U$1.2
- net SWCLK: now also JP5.8; no longer U$1.8
- net SWDIO: now also JP5.6; no longer U$1.6
- net USART_RX: now also JP5.5; no longer U$1.5
- net USART_TX: now also JP5.3; no longer U$1.3
- net WIFI_RX: now also JP5.10
- net WIFI_TX: now also JP5.9
Routing:
- net BAT+: track 12.0 -> 2.64 mm, vias 0 -> 9
- net WIFI_TX: track 26.2 -> 34.7 mm
- net NCHG: track 18.5 -> 26.7 mm, vias 2 -> 3
- net NPGOOD: track 18.6 -> 24.3 mm, vias 2 -> 3
- net WIFI_RX: track 30.0 -> 33.5 mm
- net N$8: track 0.00 -> 3.31 mm, vias 0 -> 1
- net 3.3V: track 90.4 -> 93.2 mm
- net GND: track 6.96 -> 9.75 mm, vias 98 -> 106
- net 5V: track 4.37 -> 7.13 mm, vias 0 -> 1
- net LAMP_IO: track 20.0 -> 22.7 mm, vias 2 -> 3
- net N$11: track 0.00 -> 1.97 mm, vias 0 -> 1
- net V+: track 46.0 -> 47.9 mm, vias 0 -> 1
- net POWDC: track 0.00 -> 1.71 mm, vias 0 -> 5
- net N$12: track 0.00 -> 1.56 mm, vias 0 -> 1
- net N$6: track 0.00 -> 1.40 mm, vias 0 -> 1
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- added copper zone on layer 16, net BAT+
- added copper zone on layer 16, net N$4
- added copper zone on layer 16, net POWDC
