File: wisleep_cad/wisleep/wisleep_revB.sch (EAGLE design)
At the start: 55 parts, among them IC1 STM32F10XCXT6, X1 8MHz, X2 32kHz, X3 USB-MINIB

Commit message: cad: rev B to fab
Parts:
- removed U$1: M04X2, SparkFun-Connectors:M04X2
- added C20: (no value), SparkFun-Capacitors:CAP_POL6032
- added JP5: M05X2PTH, SparkFun-Connectors:M05X2PTH
Connections:
- removed net N$26: IC1PORTB_L.PB5
- new net PB3: IC1PORTB_L.PB3
- net 3.3V: now also JP5.1; no longer U$1.1
- net 5V_ENA: now also IC1PORTB_L.PB5; no longer IC1PORTB_L.PB3
- net DBG_IO: now also JP5.4; no longer U$1.4
- net GND: now also C20.-, JP5.7; no longer U$1.7
- net N$16: now also C3.1
- net N$3: no longer C3.1
- net POWDC: now also C20.+
- net RST: now also JP5.2; no longer U$1.2
- net SWCLK: now also JP5.8; no longer U$1.8
- net SWDIO: now also JP5.6; no longer U$1.6
- net USART_RX: now also JP5.5; no longer U$1.5
- net USART_TX: now also JP5.3; no longer U$1.3
- net WIFI_RX: now also JP5.10
- net WIFI_TX: now also JP5.9
Other:
- note removed: "No plug, 1 and 2 connects"
- note removed: "With plug, 1 and 2 breaks"
- moved on the sheet: C3, C6, R6, RSENS_5V
